File: 4CH-Opto-ISO.kicad_sch (KiCad schematic)
At the start: 52 parts, among them Q1 BC847, Q2 BC847, Q3 BC847, Q4 BC847, U1 LTV-847S

Commit message: Migration to KiCad 7.0
Parts:
- C1, C2, C3, C4, C5, C6: footprint (none) -> Capacitor_SMD:C_0603_1608Metric_Pad1.08x0.95mm_HandSolder
- D1, D2, D3, D4: footprint (none) -> LED_SMD:LED_0603_1608Metric_Pad1.05x0.95mm_HandSolder
- H1, H2: footprint (none) -> MountingHole:MountingHole_3.2mm_M3_DIN965
- J1: value (none) -> IN; footprint (none) -> Connector_PinSocket_2.54mm:PinSocket_1x10_P2.54mm_Horizontal
- J2: value (none) -> IN_VT; footprint (none) -> Connector_PinSocket_2.54mm:PinSocket_1x02_P2.54mm_Horizontal
- J3: value (none) -> IN_VB; footprint (none) -> Connector_PinHeader_2.54mm:PinHeader_1x02_P2.54mm_Horizontal
- J4: value (none) -> OUT_VT; footprint (none) -> Connector_PinSocket_2.54mm:PinSocket_1x02_P2.54mm_Horizontal
- J5: value (none) -> OUT_VB; footprint (none) -> Connector_PinHeader_2.54mm:PinHeader_1x02_P2.54mm_Horizontal
- J6: value (none) -> OUT; footprint (none) -> Connector_PinHeader_2.54mm:PinHeader_1x10_P2.54mm_Horizontal
- R1, R13, R5, R9: value (none) -> 100; footprint (none) -> Resistor_SMD:R_0603_1608Metric_Pad0.98x0.95mm_HandSolder
- R10, R14, R2, R6: footprint (none) -> Resistor_SMD:R_0603_1608Metric_Pad0.98x0.95mm_HandSolder; now not fitted
- R11, R12, R15, R16, R17, R18, R19, R20, R22, R24, R26, R28, R3, R4, R7, R8: footprint (none) -> Resistor_SMD:R_0603_1608Metric_Pad0.98x0.95mm_HandSolder
- R21, R23, R25, R27: value (none) -> 0; footprint (none) -> Resistor_SMD:R_0603_1608Metric_Pad0.98x0.95mm_HandSolder
